File: 70cm_2W_PA/70cm_pa.sch (KiCad schematic (older format))
At the start: 53 parts, among them J5 Conn_01x02, U1 M68710L, U2 MIC5205YM5, U3 SN74LV1T08

Commit message: M68710L: More minor layout cleanup
Maybe it's good enough now
Parts:
- J1, J2, J6: footprint 70cm_pa:Pigtail -> 70cm_pa:Pigtail2
Changed lines of the file:
@@
 F 0 "J6" H 828 5897 50  0000 C CNN
 F 1 "~" H 828 5897 50  0000 C CNN
-F 2 "70cm_pa:Pigtail" H 900 5750 50  0001 C CNN
+F 2 "70cm_pa:Pigtail2" H 900 5750 50  0001 C CNN
 F 3 " ~" H 900 5750 50  0001 C CNN
 	1    900  5750
@@
 F 0 "J2" H 8750 1629 50  0000 L CNN
 F 1 "~" H 8750 1584 50  0000 L CNN
-F 2 "70cm_pa:Pigtail" H 8650 1700 50  0001 C CNN
+F 2 "70cm_pa:Pigtail2" H 8650 1700 50  0001 C CNN
 F 3 " ~" H 8650 1700 50  0001 C CNN
 	1    8650 1700
@@
 F 0 "J1" H 878 1847 50  0000 C CNN
 F 1 "~" H 878 1847 50  0000 C CNN
-F 2 "70cm_pa:Pigtail" H 950 1700 50  0001 C CNN
+F 2 "70cm_pa:Pigtail2" H 950 1700 50  0001 C CNN
 F 3 " ~" H 950 1700 50  0001 C CNN
 	1    950  1700
