File: 70cm_2W_PA/70cm_pa.kicad_pcb (KiCad board)
At the start: 2 copper layers, 48.3 x 48.3 mm, 53 parts, among them J5 Conn_01x02, U1 M68710L, U2 MIC5205YM5, U3 SN74LV1T08

Commit message: M68710L: More minor layout cleanup
Maybe it's good enough now
Parts:
- J1, J2, J6: footprint 70cm_pa:Pigtail -> 70cm_pa:Pigtail2
- moved R12 3.81 mm to (54.6, 55.9)
- moved R14 3.81 mm to (50.8, 55.9)
- moved R8 3.71 mm to (54.9, 66.4), turned to 180 degrees
- moved C9 2.69 mm to (56.5, 59.7), turned to 90 degrees
- moved C8 1.27 mm to (53.3, 63.5)
Routing:
- net GND: track 32.2 -> 63.1 mm, vias 357 -> 368
- net /V_supply: track 22.3 -> 25.6 mm
- net /NTC1: track 10.4 -> 7.35 mm
- net /REG_OUT: track 6.57 -> 9.53 mm
- net /V_in: track 9.48 -> 7.33 mm
- net /RF_out: track 7.70 -> 8.93 mm

Commit message: M68710L: Ready to be ordered now?
Parts:
- moved L1 1.13 mm to (64.1, 48.6), turned to 90 degrees
- moved C3 0.64 mm to (63.5, 54.0)
- moved C6 0.64 mm to (66.7, 53.0)
- moved C7 0.64 mm to (66.7, 54.9)
- moved L2 0.63 mm to (61.6, 54.0)
- moved R1 0.63 mm to (33.7, 55.2)
- moved R2 0.63 mm to (33.7, 51.4)
- moved R4 0.63 mm to (33.7, 53.3)
- moved R5 0.63 mm to (33.7, 49.5)
- moved C5 0.63 mm to (67.3, 48.6)
Routing:
- net Net-(C3-Pad1): track 10.5 -> 12.2 mm
- net GND: track 63.1 -> 64.6 mm, vias 368 -> 370
- net /PA_in: track 10.7 -> 9.76 mm
- net /V_supply: track 25.6 -> 26.6 mm
Other:
- board text added: "M68710L 70 cm PA"
- board text added: "OH2EAT 2019"
- board text removed: "M68710L 70 cm PA Tatu Peltola 2019"
